Commit message: bots joint are corrected

File: body.urdf (robot description, URDF)
Before this commit: robot robot, 3 links, 2 joints
Joints:
- removed joint BackLeg
- added joint Torso_BackLeg: type revolute, parent Torso, child BackLeg, origin xyz=1.0 0 1.0 rpy=0 0 0, axis 0 1 0, limit lower=-3.14159 upper=3.14159 effort=0.0 velocity=0.0
- joint Torso_FrontLeg: origin xyz=0 -0.5 1 rpy=0 0 0 -> xyz=2.0 0 1.0 rpy=0 0 0

Commit message: The Quadruped completed = N

File: body.urdf (robot description, URDF)
Before this commit: robot robot, 3 links, 2 joints
Links:
- added link BackLowerLeg, mass 1; collision box size=0.2 0.2 1; visual box size=0.2 0.2 1
- added link FrontLowerLeg, mass 1; collision box size=0.2 0.2 1; visual box size=0.2 0.2 1
- added link LeftLeg, mass 1; collision box size=1 0.2 0.2; visual box size=1 0.2 0.2
- added link LeftLowerLeg, mass 1; collision box size=0.2 0.2 1; visual box size=0.2 0.2 1
- added link RightLeg, mass 1; collision box size=1 0.2 0.2; visual box size=1 0.2 0.2
- added link RightLowerLeg, mass 1; collision box size=0.2 0.2 1; visual box size=0.2 0.2 1
- link BackLeg: geometry collision box size=0.2 1 0.2; visual box size=0.2 1 0.2
- link FrontLeg: geometry collision box size=0.2 1 0.2; visual box size=0.2 1 0.2
Joints:
- added joint BackLeg_BackLowerLeg: type revolute, parent BackLeg, child BackLowerLeg, origin xyz=0 -1.0 0 rpy=0 0 0, axis 0 1 0, limit lower=-3.14159 upper=3.14159 effort=0.0 velocity=0.0
- added joint FrontLeg_FrontLowerLeg: type revolute, parent FrontLeg, child FrontLowerLeg, origin xyz=0 1.0 0 rpy=0 0 0, axis 0 1 0, limit lower=-3.14159 upper=3.14159 effort=0.0 velocity=0.0
- added joint LeftLeg_LeftLowerLeg: type revolute, parent LeftLeg, child LeftLowerLeg, origin xyz=1.0 0 0 rpy=0 0 0, axis 0 1 0, limit lower=-3.14159 upper=3.14159 effort=0.0 velocity=0.0
- added joint RightLeg_RightLowerLeg: type revolute, parent RightLeg, child RightLowerLeg, origin xyz=-1.0 0 0 rpy=0 0 0, axis 0 1 0, limit lower=-3.14159 upper=3.14159 effort=0.0 velocity=0.0
- added joint Torso_LeftLeg: type revolute, parent Torso, child LeftLeg, origin xyz=0.5 0 0.5 rpy=0 0 0, axis 0 1 0, limit lower=-3.14159 upper=3.14159 effort=0.0 velocity=0.0
- added joint Torso_RightLeg: type revolute, parent Torso, child RightLeg, origin xyz=-0.5 0 0.5 rpy=0 0 0, axis 0 1 0, limit lower=-3.14159 upper=3.14159 effort=0.0 velocity=0.0
- joint Torso_BackLeg: origin xyz=1.0 0 1.0 rpy=0 0 0 -> xyz=0 -0.5 0.5 rpy=0 0 0
- joint Torso_FrontLeg: origin xyz=2.0 0 1.0 rpy=0 0 0 -> xyz=0 0.5 0.5 rpy=0 0 0

Commit message: floating on air task completed

File: body.urdf (robot description, URDF)
Before this commit: robot robot, 9 links, 8 joints
Joints:
- joint BackLeg_BackLowerLeg: axis 0 1 0 -> 1 0 0; limit lower=-3.14159 upper=3.14159 effort=0.0 velocity=0.0 -> lower=0.0 upper=1.0 effort=0.0 velocity=0.0
- joint FrontLeg_FrontLowerLeg: axis 0 1 0 -> 1 0 0; limit lower=-3.14159 upper=3.14159 effort=0.0 velocity=0.0 -> lower=0.0 upper=1.0 effort=0.0 velocity=0.0
- joint LeftLeg_LeftLowerLeg: limit lower=-3.14159 upper=3.14159 effort=0.0 velocity=0.0 -> lower=0.0 upper=1.0 effort=0.0 velocity=0.0
- joint RightLeg_RightLowerLeg: limit lower=-3.14159 upper=3.14159 effort=0.0 velocity=0.0 -> lower=0.0 upper=1.0 effort=0.0 velocity=0.0
- joint Torso_BackLeg: limit lower=-3.14159 upper=3.14159 effort=0.0 velocity=0.0 -> lower=-0.5 upper=0.5 effort=0.0 velocity=0.0; origin xyz=0 -0.5 0.5 rpy=0 0 0 -> xyz=0 -0.5 1 rpy=0 0 0
- joint Torso_FrontLeg: limit lower=-3.14159 upper=3.14159 effort=0.0 velocity=0.0 -> lower=-0.5 upper=0.5 effort=0.0 velocity=0.0; origin xyz=0 0.5 0.5 rpy=0 0 0 -> xyz=0 0.5 1 rpy=0 0 0
- joint Torso_LeftLeg: axis 0 1 0 -> 1 0 0; limit lower=-3.14159 upper=3.14159 effort=0.0 velocity=0.0 -> lower=-0.5 upper=0.5 effort=0.0 velocity=0.0; origin xyz=0.5 0 0.5 rpy=0 0 0 -> xyz=0.5 0 1 rpy=0 0 0
- joint Torso_RightLeg: axis 0 1 0 -> 1 0 0; limit lower=-3.14159 upper=3.14159 effort=0.0 velocity=0.0 -> lower=-0.5 upper=0.5 effort=0.0 velocity=0.0; origin xyz=-0.5 0 0.5 rpy=0 0 0 -> xyz=-0.5 0 1 rpy=0 0 0

Commit message: floating on air fully completed

File: body.urdf (robot description, URDF)
Before this commit: robot robot, 9 links, 8 joints
Joints:
- joint BackLeg_BackLowerLeg: limit lower=0.0 upper=1.0 effort=0.0 velocity=0.0 -> lower=-3.14159 upper=3.14159 effort=0.0 velocity=0.0
- joint FrontLeg_FrontLowerLeg: limit lower=0.0 upper=1.0 effort=0.0 velocity=0.0 -> lower=-3.14159 upper=3.14159 effort=0.0 velocity=0.0
- joint LeftLeg_LeftLowerLeg: limit lower=0.0 upper=1.0 effort=0.0 velocity=0.0 -> lower=-3.14159 upper=3.14159 effort=0.0 velocity=0.0
- joint RightLeg_RightLowerLeg: limit lower=0.0 upper=1.0 effort=0.0 velocity=0.0 -> lower=-3.14159 upper=3.14159 effort=0.0 velocity=0.0
- joint Torso_BackLeg: limit lower=-0.5 upper=0.5 effort=0.0 velocity=0.0 -> lower=-3.14159 upper=3.14159 effort=0.0 velocity=0.0
- joint Torso_FrontLeg: limit lower=-0.5 upper=0.5 effort=0.0 velocity=0.0 -> lower=-3.14159 upper=3.14159 effort=0.0 velocity=0.0
- joint Torso_LeftLeg: limit lower=-0.5 upper=0.5 effort=0.0 velocity=0.0 -> lower=-3.14159 upper=3.14159 effort=0.0 velocity=0.0
- joint Torso_RightLeg: limit lower=-0.5 upper=0.5 effort=0.0 velocity=0.0 -> lower=-3.14159 upper=3.14159 effort=0.0 velocity=0.0

Commit message: standingOn2Feet

File: body.urdf (robot description, URDF)
Before this commit: robot robot, 9 links, 8 joints
Links:
- removed link BackLeg
- removed link BackLowerLeg
- removed link FrontLeg
- removed link FrontLowerLeg
- removed link LeftLeg
- removed link LeftLowerLeg
- removed link RightLeg
- removed link RightLowerLeg
- added link LeftFoot, mass 1; collision box size=0.15 0.4 0.1; visual box size=0.15 0.4 0.1
- added link LeftShin, mass 1; collision box size=0.12 0.12 0.6; visual box size=0.12 0.12 0.6
- added link LeftThigh, mass 1; collision box size=0.15 0.15 0.6; visual box size=0.15 0.15 0.6
- added link RightFoot, mass 1; collision box size=0.15 0.4 0.1; visual box size=0.15 0.4 0.1
- added link RightShin, mass 1; collision box size=0.12 0.12 0.6; visual box size=0.12 0.12 0.6
- added link RightThigh, mass 1; collision box size=0.15 0.15 0.6; visual box size=0.15 0.15 0.6
- link Torso: geometry collision box size=0.4 0.2 0.8; visual box size=0.4 0.2 0.8
Joints:
- removed joint BackLeg_BackLowerLeg
- removed joint FrontLeg_FrontLowerLeg
- removed joint LeftLeg_LeftLowerLeg
- removed joint RightLeg_RightLowerLeg
- removed joint Torso_BackLeg
- removed joint Torso_FrontLeg
- removed joint Torso_LeftLeg
- removed joint Torso_RightLeg
- added joint LeftShin_LeftFoot: type revolute, parent LeftShin, child LeftFoot, origin xyz=0 0 -0.6 rpy=0 0 0, axis 1 0 0, limit lower=-3.14159 upper=3.14159 effort=0.0 velocity=0.0
- added joint LeftThigh_LeftShin: type revolute, parent LeftThigh, child LeftShin, origin xyz=0 0 -0.6 rpy=0 0 0, axis 1 0 0, limit lower=-3.14159 upper=3.14159 effort=0.0 velocity=0.0
- added joint RightShin_RightFoot: type revolute, parent RightShin, child RightFoot, origin xyz=0 0 -0.6 rpy=0 0 0, axis 1 0 0, limit lower=-3.14159 upper=3.14159 effort=0.0 velocity=0.0
- added joint RightThigh_RightShin: type revolute, parent RightThigh, child RightShin, origin xyz=0 0 -0.6 rpy=0 0 0, axis 1 0 0, limit lower=-3.14159 upper=3.14159 effort=0.0 velocity=0.0
- added joint Torso_LeftThigh: type revolute, parent Torso, child LeftThigh, origin xyz=0.1 0 1.1 rpy=0 0 0, axis 1 0 0, limit lower=-3.14159 upper=3.14159 effort=0.0 velocity=0.0
- added joint Torso_RightThigh: type revolute, parent Torso, child RightThigh, origin xyz=-0.1 0 1.1 rpy=0 0 0, axis 1 0 0, limit lower=-3.14159 upper=3.14159 effort=0.0 velocity=0.0

Commit message: biped with arms completed finally

File: body.urdf (robot description, URDF)
Before this commit: robot robot, 7 links, 6 joints
Links:
- added link LeftLowerArm, mass 1; collision box size=0.3 0.1 0.1; visual box size=0.3 0.1 0.1
- added link LeftUpperArm, mass 1; collision box size=0.3 0.1 0.1; visual box size=0.3 0.1 0.1
- added link RightLowerArm, mass 1; collision box size=0.3 0.1 0.1; visual box size=0.3 0.1 0.1
- added link RightUpperArm, mass 1; collision box size=0.3 0.1 0.1; visual box size=0.3 0.1 0.1
Joints:
- added joint LeftUpperArm_LeftLowerArm: type revolute, parent LeftUpperArm, child LeftLowerArm, origin xyz=0.3 0 0 rpy=0 0 0, axis 0 1 0, limit lower=-3.14159 upper=3.14159 effort=0.0 velocity=0.0
- added joint RightUpperArm_RightLowerArm: type revolute, parent RightUpperArm, child RightLowerArm, origin xyz=-0.3 0 0 rpy=0 0 0, axis 0 1 0, limit lower=-3.14159 upper=3.14159 effort=0.0 velocity=0.0
- added joint Torso_LeftUpperArm: type revolute, parent Torso, child LeftUpperArm, origin xyz=0.2 0 1.9 rpy=0 0 0, axis 0 1 0, limit lower=-3.14159 upper=3.14159 effort=0.0 velocity=0.0
- added joint Torso_RightUpperArm: type revolute, parent Torso, child RightUpperArm, origin xyz=-0.2 0 1.9 rpy=0 0 0, axis 0 1 0, limit lower=-3.14159 upper=3.14159 effort=0.0 velocity=0.0
