Commit message: multiple robots task completed

File: body0.urdf (robot description, URDF)
Before this commit: robot robot, 9 links, 8 joints
Joints:
- joint BackLeg_BackLowerLeg: axis 0 1 0 -> 1 0 0
- joint FrontLeg_FrontLowerLeg: axis 0 1 0 -> 1 0 0
- joint Torso_BackLeg: axis 0 1 0 -> 1 0 0; origin xyz=0 -0.5 0.5 rpy=0 0 0 -> xyz=0.0 -0.5 0.5 rpy=0 0 0
- joint Torso_FrontLeg: axis 0 1 0 -> 1 0 0; origin xyz=0 0.5 0.5 rpy=0 0 0 -> xyz=0.0 0.5 0.5 rpy=0 0 0
